File: hardware/falloutbadge.kicad_sch (KiCad schematic)
At the start: 0 parts

Commit message: schematic with stm32
Parts:
- added AE1: Antenna, symbol Device:Antenna
- added BZ1: Buzzer, Buzzer_Beeper:Buzzer_TDK_PS1240P02BT_D12.2mm_H6.5mm, symbol Device:Buzzer
- added C1, C15, C16, C3, C32, C35, C42, C45, C47, C54: 100nF, Capacitor_SMD:C_0402_1005Metric, symbol Device:C
- added C10, C14: 68pF, symbol Device:C
- added C11, C13: 1nF, symbol Device:C
- added C12, C9: 10pF, symbol Device:C
- added C17, C18, C19: 4.7uF, Capacitor_SMD:C_0603_1608Metric, symbol Device:C
- added C2: 68pF, Capacitor_SMD:C_0402_1005Metric, symbol Device:C
- added C20, C22: 2.2pF, Capacitor_SMD:C_0402_1005Metric, symbol Device:C
- added C21, C23, C24, C25, C26, C27, C28, C29, C30, C31: 1uF, Capacitor_SMD:C_0603_1608Metric, symbol Device:C
- added C37, C38: 20pF, symbol Device:C
- added C39: 100uF, Capacitor_SMD:C_0805_2012Metric, symbol Device:C
- added C4: 100pF, symbol Device:C
- added C49, C51, C55: 10uF, Capacitor_SMD:C_0603_1608Metric, symbol Device:C
- added C5: 1uF, symbol Device:C
- added C6: 47nF, Capacitor_SMD:C_0402_1005Metric, symbol Device:C
- added C7: 220nF, Capacitor_SMD:C_0402_1005Metric, symbol Device:C
- added C8: 100nF, symbol Device:C
- added D1, D17, D18: LED, LED_SMD:LED_0603_1608Metric, symbol Device:LED
- added D2, D3, D4: D, Diode_SMD:D_SOD-123, symbol Diode:MBR0530
- added D5: D, symbol Device:D
- added D6: RED, LED_SMD:LED_0603_1608Metric, symbol Device:LED
- added D7: GREEN, LED_SMD:LED_0603_1608Metric, symbol Device:LED
- added D8: SK6812SIDE-A-RVS, falloutbadge:LED-SMD_4P-L4.0-W1.6-L, symbol LED:SK6812
- added FB2: BLM18AG601SN1D, Resistor_SMD:R_0603_1608Metric, symbol Device:FerriteBead
- added J1: USB_C_Receptacle_USB2.0_16P, Connector_USB:USB_C_Receptacle_HRO_TYPE-C-31-M-12, symbol Connector:USB_C_Receptacle_USB2.0_16P
- added J2: E-INK, falloutbadge:FPC-SMD_24P-P0.50_05B20U24P, symbol Connector_Generic:Conn_01x24
- added J3: Conn_01x03, Connector_PinHeader_2.54mm:PinHeader_1x03_P2.54mm_Vertical_SMD_Pin1Left, symbol Connector_Generic:Conn_01x03
- added J4: LiPo, Connector_JST:JST_PH_S2B-PH-K_1x02_P2.00mm_Horizontal, symbol Connector_Generic:Conn_01x02
- added J5: Conn_02x03, Connector_PinSocket_2.54mm:PinSocket_2x03_P2.54mm_Vertical, symbol Connector_Generic:Conn_02x03_Counter_Clockwise
- added L1: 2.0uH, falloutbadge:antenna28, symbol Device:L
- added L2: 68uH, Inductor_SMD:L_APV_ANR4018, symbol Device:L
- added L3: 47nH, symbol Device:L
- added L4: 6.8uH, symbol Device:L
- added Q1: NMOS, Package_TO_SOT_SMD:SOT-323_SC-70, symbol Simulation_SPICE:NMOS
- added Q2: AO3400, Package_TO_SOT_SMD:TSOT-23, symbol Device:Q_NPN
- added R1, R9: 4.7k, Resistor_SMD:R_0402_1005Metric, symbol Device:R
- added R10: 10k, Resistor_SMD:R_0603_1608Metric, symbol Device:R
- added R11: 0.47R, Resistor_SMD:R_0603_1608Metric, symbol Device:R
- added R12, R3: 5.1k, Resistor_SMD:R_0402_1005Metric, symbol Device:R
- added R13, R2: 10k, symbol Device:R
- added R14: 330R, Resistor_SMD:R_0603_1608Metric, symbol Device:R
- added R15, R16: 1k, Resistor_SMD:R_0402_1005Metric, symbol Device:R
- added R17: 3.3k, Resistor_SMD:R_0402_1005Metric, symbol Device:R
- added R4, R6: 5.1k, symbol Device:R
- added R5: 47R, Resistor_SMD:R_0603_1608Metric, symbol Device:R
- added R7: 100R, symbol Device:R
- added R8: 330R, symbol Device:R
- added SW1: SW_Push, symbol Switch:SW_Push
- added SW10, SW7, SW8, SW9: SW_Push, Button_Switch_THT:SW_PUSH_1P1T_6x3.5mm_H4.3_APEM_MJTP1243, symbol Switch:SW_Push
- added SW3, SW4, SW5, SW6: SW_Push, Button_Switch_THT:SW_PUSH-12mm_Wuerth-430476085716, symbol Switch:SW_Push
- added T1: BALFLB-WL-09D3, easyeda2kicad:CSPG-8_L2.1-W1.8_BALFHB-WL-03D3, symbol easy:BALFLB-WL-09D3
- added TP1, TP2, TP3, TP4, TP5, TP6, TP7, TP8: TestPoint, TestPoint:TestPoint_Pad_D1.0mm, symbol Connector:TestPoint
- added U1: NT3H2111-2211, falloutbadge:QFN8P50_160X160X50L40X20N, symbol falloutbadge:NT3H2111_2211
- added U10: STM32WLE5CCUx, Package_DFN_QFN:QFN-48-1EP_7x7mm_P0.5mm_EP5.6x5.6mm, symbol MCU_ST_STM32WL:STM32WLE5CCUx
- added U2: BGS12WN6E6327, Package_LGA:Infineon_PG-TSNP-6-10_0.7x1.1mm_0.7x1.1mm_P0.4mm, symbol RF_Switch:BGS12WN6E6327
- added U3: CH9102F, Package_DFN_QFN:QFN-24-1EP_4x4mm_P0.5mm_EP2.6x2.6mm, symbol Interface_USB:CH9102F
- added U5: USBLC6-2SC6, Package_TO_SOT_SMD:SOT-23-6, symbol Power_Protection:USBLC6-2SC6
- added U6: TP4056, Package_SO:SOIC-8-1EP_3.9x4.9mm_P1.27mm_EP2.41x3.3mm_ThermalVias, symbol Battery_Management:TP4056-42-ESOP8
- added U8: AP2112K-3.3, Package_TO_SOT_SMD:SOT-23-5, symbol Regulator_Linear:AP2112K-3.3
- added Y1: 32MHz, Crystal:Crystal_SMD_3225-4Pin_3.2x2.5mm, symbol Device:Crystal_GND24
Connections:
- new net: C24.2, J2.19 (Pin_19)
- new net: C14.1, C20.1, L4.1
- new net: C14.2, U2.5 (RFIN)
- new net: R17.1, U6.2 (PROG)
- new net: C8.2, R2.2, SW1.2, U10.18 (NRST)
- new net: C11.1, C9.1, R7.1, U2.6 (CTRL)
- new net: C2.2, C6.2, L3.1, U10.24 (VR_PA)
- new net: FB2.1, J1.S1 (SHIELD)
- new net: C4.2, T1.A1 (RFO_in)
- new net: C10.2, T1.C1 (RFO_out)
- new net: T1.C3 (RFI_in), U2.1 (RF2)
- new net: C23.2, J2.18 (Pin_18)
- new net: AE1.1 (A), C22.1, L4.2
- new net: C38.2, U10.27 (OSC_OUT), Y1.3
- new net: C30.2, J2.4 (Pin_4)
- new net: C1.1, U10.29 (VDDRF1V55)
- new net: D7.1 (K), R16.1
- new net: C18.1, D2.2 (A), D3.1 (K)
- new net: C10.1, U2.3 (RF1)
- new net: D1.2 (A), R5.2
- new net: D5.2 (A), J1.A4 (VBUS), J1.A9 (VBUS), J1.B4 (VBUS), J1.B9 (VBUS)
- new net: D17.2 (A), R6.2
- new net: C18.2, D4.2 (A), L2.2, Q1.1 (D)
- new net: C25.2, J2.20 (Pin_20)
- new net: C27.2, J2.22 (Pin_22)
- new net: C29.2, J2.24 (Pin_24)
- new net: C31.2, J2.5 (Pin_5)
- new net: D6.1 (K), R15.1
- new net: C7.1, R5.1, U1.7 (VOUT)
- new net: Q2.B, R8.2
- new net: L1.2, U1.1 (LA)
- new net: J1.A5 (CC1), R12.1
- new net: J1.A6 (D+), J1.B6 (D+), U5.3 (I/O2)
- new net: J1.A7 (D-), J1.B7 (D-), U5.1 (I/O1)
- new net: J1.B5 (CC2), R3.1
- new net: D18.1 (K), U3.14 (TXS/GPIO0)
- new net: D18.2 (A), R4.2
- new net: C37.2, U10.26 (OSC_IN), Y1.1
- new net: R16.2, U6.6 (~{STDBY})
- new net: R15.2, U6.7 (~{CHRG})
- new net: D17.1 (K), U3.13 (RXS/GPIO1)
- new net: BZ1.2 (-), Q2.C
- new net +3V3: BZ1.1 (+), C12.1, C13.1, C15.1, C16.1, C17.1, C19.1, C21.2, C3.1, C32.1, C35.1, C54.1, C55.2, D6.2 (A), D7.2 (A), J2.15 (Pin_15), J2.16 (Pin_16), J5.1 (Pin_1), L2.1, R1.1, R2.1, R4.1, R6.1, R9.1, TP3.1, U1.6 (VDD), U10.11 (VDD), U10.25 (VDDPA), U10.28 (VDDRF), U10.37 (VBAT), U10.41 (VDDA), U10.44 (VDD), U10.46 (VDDSMPS), U2.4 (VDD), U3.5 (VIO), U3.6 (V3), U8.5 (VOUT)
- new net +BATT: C49.2, C51.1, J4.1 (Pin_1), TP7.1, U6.5 (BAT), U8.1 (VIN), U8.3 (EN)
- new net BUSY: J2.9 (Pin_9), U10.4 (PB6)
- new net CS: J2.12 (Pin_12), U10.32 (PB12)
- new net CTRL: R13.1, R7.2, U10.2 (PB4)
- new net D+: U3.3 (D+), U5.4 (I/O2)
- new net D-: U3.4 (D-), U5.6 (I/O1)
- new net DC: J2.11 (Pin_11), U10.6 (PB8)
- new net GDR: J2.2 (Pin_2), Q1.2 (G), R10.1
- new net GND: C1.2, C11.2, C12.2, C13.2, C15.2, C16.2, C17.2, C19.2, C2.1, C20.2, C21.1, C22.2, C23.1, C24.1, C25.1, C26.1, C27.1, C28.1, C29.1, C3.2, C30.1, C31.1, C32.2, C35.2, C37.1, C38.1, C39.1, C42.2, C45.2, C47.2, C49.1, C5.1, C51.2, C54.2, C55.1, C6.1, C7.2, C8.1, C9.2, D1.1 (K), D2.1 (K), D8.1 (VSS), FB2.2, J1.A1 (GND), J1.A12 (GND), J1.B1 (GND), J1.B12 (GND), J2.17 (Pin_17), J2.8 (Pin_8), J3.2 (Pin_2), J4.2 (Pin_2), J5.2 (Pin_2), Q2.E, R10.2, R11.2, R12.2, R13.2, R17.2, R3.2, SW1.1, SW10.2, SW3.2, SW4.2, SW5.2, SW6.2, SW7.2, SW8.2, SW9.2, T1.B1 (GND2), T1.B2 (GND3), T1.C2 (GND1), TP4.1, TP6.1, TP8.1, U1.2 (VSS), U10.45 (VFBSMPS), U10.48 (VSSSMPS), U10.49 (VSS), U2.2 (GND), U3.2 (GND), U3.25 (GND), U5.2 (GND), U6.1 (TEMP), U6.3 (GND), U6.9 (EPAD), U8.2 (GND), Y1.2, Y1.4
- new net LB: L1.1, U1.8 (LB)
- new net PA0: R8.1, U10.7 (PA0)
- new net PA1: SW3.1, U10.8 (PA1)
- new net PA15: R14.1, U10.43 (PA15)
- new net PA2: SW4.1, U10.9 (PA2)
- new net PA3: SW5.1, U10.10 (PA3)
- new net PA4: SW6.1, U10.12 (PA4)
- new net PA5: SW7.1, U10.13 (PA5)
- new net PA6: SW8.1, U10.14 (PA6)
- new net PA7: SW9.1, U10.15 (PA7)
- new net PA8: SW10.1, U10.16 (PA8)
- new net PB0: J5.6 (Pin_6), U10.30 (PB0)
- new net PB2: J5.5 (Pin_5), U10.31 (PB2)
- new net PREVGH: C26.2, D4.1 (K), J2.21 (Pin_21)
- new net PREVGL: C28.2, D3.2 (A), J2.23 (Pin_23)
- new net RESE: J2.3 (Pin_3), Q1.3 (S), R11.1
- new net RFI_N: T1.A2 (RFI_N_out), U10.21 (RFI_N)
- new net RFI_P: T1.A3 (RFI_P_out), U10.20 (RFI_P)
- new net RFO_HP: C4.1, L3.2, U10.23 (RFO_HP)
- new net RST: J2.10 (Pin_10), U10.5 (PB7)
- new net RXD: U10.17 (PA9), U3.20 (RXD)
- new net SCL: J5.4 (Pin_4), R9.2, TP1.1, U1.3 (SCL), U10.35 (PA12)
- new net SDA: J5.3 (Pin_3), R1.2, TP2.1, U1.5 (SDA), U10.34 (PA11)
- new net SPI_MOSI: J2.14 (Pin_14), U10.3 (PB5)
- new net SPI_SCK: J2.13 (Pin_13), U10.1 (PB3)
- new net SWCLK: J3.1 (Pin_1), U10.42 (PA14)
- new net SWDIO: J3.3 (Pin_3), U10.36 (PA13)
- new net TXD: U10.33 (PA10), U3.21 (TXD)
- new net VBUS: C39.2, C42.1, C45.1, C47.1, C5.2, D5.1 (K), D8.3 (VDD), TP5.1, U3.7 (VDD5), U3.8 (VBUS), U5.5 (VBUS), U6.4 (V_{CC}), U6.8 (CE)
- new net led/DIN: R14.2
- new net led3/DOUT: D8.2 (DIN)
- no-connect marks 0 -> 26
Other:
- added sheet led (led.kicad_sch)
- added sheet led1 (led.kicad_sch)
- added sheet led2 (led.kicad_sch)
- added sheet led3 (led.kicad_sch)
- note added: "17dBm to stay under the limit of 19dBm"
- note added: "2.9""
- note added: "AP2112K"
- note added: "Back light"
- note added: "Buttons"
- note added: "Buzzer"
- note added: "CHECK"
- note added: "CN470 (470-510 MHz)"
- note added: "E-Paper Display"
- note added: "Large"
- note added: "LiPo"
- note added: "NFC"
- note added: "NeoPixels"
- note added: "RF Output"
- note added: "SAO"
- note added: "STM32 MCU"
- note added: "SWD"
- note added: "Small"
- note added: "TP4056"
- note added: "Test Points"
- note added: "add more"
- note added: "check footprint"
- note added: "for ~360mA charge current"
