File: hardware/falloutbadge.kicad_sch (KiCad schematic)
At the start: 108 parts, among them J1 LiPo, J3 USB_C_Receptacle_USB2.0_16P, J4 E-INK, J5 Conn_01x03, Q2 NMOS, Q3 AO3400A, SW1 SW_Push, SW2 SW_Push, SW3 SW_Push, SW4 SW_Push, SW5 SW_Push, T1 BALFLB-WL-09D3, U1 CH592F, U2 STM32WLE5CCUx, U3 CH9102F, U4 USBLC6-2SC6, U5 TP4056, U6 BGS12SN6, U7 AP2112K-3.3, Y1 32MHz, Y2 32MHz

Commit message: vddrf1v5 and smps, + uart fix
Parts:
- added C12: 100nF, Capacitor_SMD:C_0402_1005Metric, symbol Device:C
Connections:
- net +3V3: no longer C23.1, U2.45 (VFBSMPS), U3.6 (V3)
- net GND: now also C12.1
- net VFBSMPS: now reaches C16.1, U2.29 (VDDRF1V55)
- net VFBSMPS: now also U2.45 (VFBSMPS), C12.2
- new net: C23.1, U3.6 (V3)
Other:
- moved on the sheet: C23, C34

Commit message: final fixes
Parts:
- removed U5: TP4056, Package_SO:SOIC-8-1EP_3.9x4.9mm_P1.27mm_EP2.41x3.3mm_ThermalVias, symbol Battery_Management:TP4056-42-ESOP8
- added U5: CH340C, Package_SO:SOIC-16_3.9x9.9mm_P1.27mm, symbol Interface_USB:CH340C
- added U8: TP4056-42-ESOP8, Package_SO:SOIC-8-1EP_3.9x4.9mm_P1.27mm_EP2.41x3.3mm_ThermalVias, symbol Battery_Management:TP4056-42-ESOP8
- AE2: LCSC C718845 -> (none); LCSC Part # (none) -> C718845
- AE3: footprint antenna:ANT-F-1-2.4G-1.6mmFR4-WCH -> antenna:ANT-F-1-2.4G-0.8mmFR4-WCH; now left out of the parts list
- BZ1: LCSC C76871 -> (none); LCSC Part # (none) -> C76871
- C1, C12, C14, C15, C16, C17, C18, C2, C23, C34, C4, C47, C49, C53, C54: LCSC Part # (none) -> C1525
- C10, C48: LCSC Part # (none) -> C69335
- C11, C21, C50, C52: LCSC Part # (none) -> C52923
- C19: LCSC Part # (none) -> C19702; now left out of the parts list
- C20, C22: footprint Capacitor_SMD:C_0603_1608Metric -> Capacitor_SMD:C_1206_3216Metric; LCSC Part # (none) -> C12881
- C24, C27, C28, C29, C30, C31, C32, C33: LCSC Part # (none) -> C15849
- C25, C26: LCSC C15849 -> (none); LCSC Part # (none) -> C15849
- C3: LCSC Part # (none) -> C92361
- C35, D9, R14: now not fitted; now left out of the parts list
- C36: LCSC C85934 -> (none); LCSC Part # (none) -> C85934
- C37: LCSC C161156 -> (none); LCSC Part # (none) -> C389103
- C38, C39: LCSC C782046 -> (none); LCSC Part # (none) -> C782046
- C40, C44: LCSC C1523 -> (none); LCSC Part # (none) -> C1523
- C41: LCSC C14441 -> (none); LCSC Part # (none) -> C389103
- C42, C46: value 10uF -> 4.7uF; LCSC Part # (none) -> C19666
- C5, C6: value 20pF -> 6.8pF; LCSC Part # (none) -> C1576
- C7: LCSC Part # (none) -> C126529
- C8: LCSC Part # (none) -> C389103
- C9: LCSC Part # (none) -> C23630
- D1, D2, D3: value D -> MBR0530; LCSC C77336 -> (none); LCSC Part # (none) -> C77336
- D4: footprint (none) -> Diode_SMD:D_SOD-123F; LCSC Part # (none) -> C2892326
- D7: LCSC Part # (none) -> C84269
- D8: value GREEN -> NOT RED; LCSC Part # (none) -> C84256
- FB1: footprint Resistor_SMD:R_0603_1608Metric -> Inductor_SMD:L_0805_2012Metric; LCSC C19330 -> (none); LCSC Part # (none) -> C1017
- J1: LCSC Part # (none) -> C173752
- J3: LCSC C3020560 -> (none); LCSC Part # (none) -> C3020560
- J4: LCSC C5362165 -> (none); LCSC Part # (none) -> C5362165
- J5: now not fitted
- L1: value 47nH -> 68nH; LCSC Part # (none) -> C108965
- L3: footprint Inductor_SMD:L_APV_ANR4018 -> Inductor_SMD:L_Changjiang_FNR6028S; LCSC Part # (none) -> C168045
- L6: footprint Inductor_SMD:L_0402_1005Metric -> Inductor_SMD:L_1210_3225Metric; LCSC Part # (none) -> C354558
- Q2: value NMOS -> Si1308EDL; LCSC C7603347 -> (none); LCSC Part # (none) -> C7603347
- Q3: LCSC C20917 -> (none); LCSC Part # (none) -> C20917
- R1, R4: LCSC Part # (none) -> C25744
- R12, R13: value 1k -> 330R; LCSC Part # (none) -> C208861
- R15: LCSC Part # (none) -> C25890
- R16, R17: LCSC C25076 -> (none); LCSC Part # (none) -> C25076
- R2: LCSC Part # (none) -> C208861
- R6: footprint Resistor_SMD:R_0603_1608Metric -> Resistor_SMD:R_0402_1005Metric; LCSC Part # (none) -> C25744
- R7: footprint Resistor_SMD:R_0603_1608Metric -> Resistor_SMD:R_0402_1005Metric; LCSC Part # (none) -> C2089288
- R8, R9: LCSC Part # (none) -> C25905
- SW1: footprint Button_Switch_SMD:SW_Push_SPST_NO_Alps_SKRK -> Button_Switch_SMD:SW_SPST_TS-1088-xR025; LCSC Part # (none) -> C720477
- SW2, SW3, SW4, SW5: footprint Button_Switch_THT:SW_PUSH-12mm_Wuerth-430476085716 -> Button_Switch_THT:SW_PUSH-12mm
- T1: LCSC C5350027 -> (none); LCSC Part C5350027 -> (none); LCSC Part # (none) -> C5350027
- U1: LCSC C39831287 -> (none); LCSC Part # (none) -> C39831287
- U2: LCSC C2888218 -> (none); LCSC Part # (none) -> C2888218
- U3: LCSC C2858418 -> (none); LCSC Part # (none) -> C2858418
- U4: LCSC C2687116 -> (none); LCSC Part # (none) -> C2687116
- U6: LCSC C114953 -> (none); LCSC Part # (none) -> C114953
- U7: LCSC C23380830 -> (none); LCSC Part # (none) -> C23380830
- Y1: LCSC C5441424 -> (none); LCSC Part # (none) -> C5441424
- Y2: LCSC C9009 -> (none); LCSC Part # (none) -> C9009
Connections:
- net +3V3: now also J4.10 (Pin_10), J4.9 (Pin_9); no longer J4.15 (Pin_15), J4.16 (Pin_16)
- net +BATT: now also U8.5 (BAT)
- net BUSY: now also J4.16 (Pin_16), U2.10 (PA3); no longer J4.9 (Pin_9), U2.7 (PA0)
- net CS: now also J4.13 (Pin_13), U2.7 (PA0); no longer J4.12 (Pin_12), U2.10 (PA3)
- net DC: now also J4.14 (Pin_14), U2.8 (PA1); no longer J4.11 (Pin_11), U2.9 (PA2)
- net GDR: now also J4.23 (Pin_23); no longer J4.2 (Pin_2)
- net GND: now also U8.1 (TEMP), U8.3 (GND), U8.9 (EPAD)
- net PREVGH: now also J4.4 (Pin_4); no longer J4.21 (Pin_21)
- net PREVGL: now also J4.2 (Pin_2); no longer J4.23 (Pin_23)
- net RESE: now also J4.22 (Pin_22); no longer J4.3 (Pin_3)
- net RST: now also J4.15 (Pin_15), U2.9 (PA2); no longer J4.10 (Pin_10), U2.8 (PA1)
- net SPI_MOSI: now also J4.11 (Pin_11); no longer J4.14 (Pin_14)
- net SPI_SCK: now also J4.12 (Pin_12); no longer J4.13 (Pin_13)
- net VBUS: now also U8.4 (V_{CC}), U8.8 (CE)
- net at C28.2: now also J4.6 (Pin_6); no longer J4.19 (Pin_19)
- net at R15.1: now also U8.2 (PROG)
- net at C27.2: now also J4.7 (Pin_7); no longer J4.18 (Pin_18)
- net at C25.2: now also J4.21 (Pin_21); no longer J4.4 (Pin_4)
- net at J4.1 (Pin_1): now also C33.2
- net at J4.20 (Pin_20): now also C26.2; no longer C29.2
- net at C31.2: now also J4.3 (Pin_3); no longer J4.22 (Pin_22)
- net at J4.24 (Pin_24): no longer C33.2
- net at J4.5 (Pin_5): now also C29.2; no longer C26.2
- net at R13.2: now also U8.6 (~{STDBY})
- net at R12.2: now also U8.7 (~{CHRG})
Other:
- note added: "2.7""
- note added: "for ~300mA charge current"
- note removed: "2.9""
- note removed: "check"
- note removed: "for ~360mA charge current"
- moved on the sheet: D1, D2, D3

Commit message: assign lcsc parts and flip eink
Parts:
- J4: footprint falloutbadge:FPC-SMD_24P-P0.50_05B20U24P -> Connector_FFC-FPC:TE_2-1734839-4_1x24-1MP_P0.5mm_Horizontal
- SW2, SW3, SW4, SW5: LCSC Part # (none) -> C87494
Changed lines of the file:
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@@
 			)
 		)
+		(property "LCSC Part #" "C87494"
+			(at 279.4 229.87 0)
+			(effects
+				(font
+					(size 1.27 1.27)
+				)
+				(hide yes)
+			)
+		)
 		(pin "1"
 		)
@@
 			)
 		)
-		(property "Footprint" "falloutbadge:FPC-SMD_24P-P0.50_05B20U24P"
+		(property "Footprint" "Connector_FFC-FPC:TE_2-1734839-4_1x24-1MP_P0.5mm_Horizontal"
 			(at 245.11 240.03 0)
 			(effects
@@
 			)
 		)
+		(property "LCSC Part #" "C87494"
+			(at 279.4 209.55 0)
+			(effects
+				(font
+					(size 1.27 1.27)
+				)
+				(hide yes)
+			)
+		)
 		(pin "1"
 		)
@@
 			)
 		)
+		(property "LCSC Part #" "C87494"
+			(at 279.4 219.71 0)
+			(effects
+				(font
+					(size 1.27 1.27)
+				)
+				(hide yes)
+			)
+		)
 		(pin "1"
 		)
@@
 			(at 279.4 240.03 0)
 			(effects
+				(font
+					(size 1.27 1.27)
+				)
+				(hide yes)
+			)
+		)
+		(property "LCSC Part #" "C87494"
+			(at 279.4 240.03 0)
+			(effects

Commit message: add v2 w/o lora
Parts:
- removed AE2: Antenna, Connector_PinHeader_2.54mm:PinHeader_1x01_P2.54mm_Vertical, symbol Device:Antenna
- removed AE3: Antenna_Shield, antenna:ANT-F-1-2.4G-0.8mmFR4-WCH, symbol Device:Antenna_Shield
- removed C17, C18, C23, C34, C49, C53, C54: 100nF, Capacitor_SMD:C_0402_1005Metric, symbol Device:C
- removed C35: 100uF, symbol Device:C
- removed C36: 100pF, Capacitor_SMD:C_0201_0603Metric, symbol Device:C
- removed C37, C41: 68pF, Capacitor_SMD:C_0402_1005Metric, symbol Device:C
- removed C38, C39: 10pF, Capacitor_SMD:C_0402_1005Metric, symbol Device:C
- removed C40, C44: 1nF, Capacitor_SMD:C_0402_1005Metric, symbol Device:C
- removed C43, C45: 2.2pF, Capacitor_SMD:C_0402_1005Metric, symbol Device:C
- removed C48: 4.7uF, Capacitor_SMD:C_0603_1608Metric, symbol Device:C
- removed C50, C52: 1uF, Capacitor_SMD:C_0402_1005Metric, symbol Device:C
- removed C51: NC, Capacitor_SMD:C_0402_1005Metric, symbol Device:C
- removed C7: 47nF, Capacitor_SMD:C_0402_1005Metric, symbol Device:C
- removed D9: SK6812, footprints:LED-SMD_4P-L4.0-W1.6-L, symbol LED:SK6812
- removed L1: 68nH, Inductor_SMD:L_0402_1005Metric, symbol Device:L
- removed L4: 6.8uH, Inductor_SMD:L_0402_1005Metric, symbol Device:L
- removed R1: 10k, Resistor_SMD:R_0402_1005Metric, symbol Device:R
- removed R14: 330R, symbol Device:R
- removed R16, R17: 100R, Resistor_SMD:R_0402_1005Metric, symbol Device:R
- removed T1: BALFLB-WL-09D3, falloutbadge:CSPG-8_L2.1-W1.8_BALFHB-WL-03D3, symbol easy:BALFLB-WL-09D3
- removed TP7: CTRL, TestPoint:TestPoint_Pad_D1.0mm, symbol Connector:TestPoint
- removed U2: STM32WLE5CCUx, footprints:UFQFPN-48_L7.0-W7.0-P0.50-BL-EP5.6, symbol MCU_ST_STM32WL:STM32WLE5CCUx
- removed U3: CH9102F, Package_DFN_QFN:QFN-24-1EP_4x4mm_P0.5mm_EP2.6x2.6mm, symbol Interface_USB:CH9102F
- removed U5: CH340C, Package_SO:SOIC-16_3.9x9.9mm_P1.27mm, symbol Interface_USB:CH340C
- removed U6: BGS12SN6, Package_LGA:Infineon_PG-TSNP-6-10_0.7x1.1mm_0.7x1.1mm_P0.4mm, symbol RF_Switch:BGS12WN6E6327
- added AE2: Antenna_Shield, antenna:ANT-F-1-2.4G-1.6mmFR4-WCH, symbol Device:Antenna_Shield
- added C10, C13, C3, C9: 100nF, Capacitor_SMD:C_0402_1005Metric, symbol Device:C
- added C2: 33pF, Capacitor_SMD:C_0402_1005Metric, symbol Device:C
- added C7: 10uF, symbol Device:C_Polarized
- added D1, D12, D13, D14, D15, D16, D2, D20, D21, D4, D5, D7: SK6812, footprints:LED-SMD_4P-L4.0-W1.6-L, symbol LED:SK6812
- added H1, H2: MountingHole, MountingHole:MountingHole_2.2mm_M2_DIN965_Pad, symbol Mechanical:MountingHole_Pad
- added J1: Conn_02x03, Connector_PinHeader_2.54mm:PinHeader_1x06_P2.54mm_Vertical, symbol Connector_Generic:Conn_02x03_Counter_Clockwise
- added R2, R6: 10k, Resistor_SMD:R_0402_1005Metric, symbol Device:R
- added R3, R7: 1k, Resistor_SMD:R_0402_1005Metric, symbol Device:R
- added R5: 27.4R, Resistor_SMD:R_0402_1005Metric, symbol Device:R
- added R8: 330R, Resistor_SMD:R_0402_1005Metric, symbol Device:R
- added SW10, SW7, SW8, SW9: SW_Push, Button_Switch_THT:SW_PUSH_6mm, symbol Switch:SW_Push
- added SW2: BOOTSEL, Button_Switch_SMD:SW_Push_SPST_NO_Alps_SKRK, symbol Switch:SW_Push
- added U1: W25Q32JVSS, Package_SO:SOIC-8_5.3x5.3mm_P1.27mm, symbol Memory_Flash:W25Q32JVSS
- added U2: RP2040, Package_DFN_QFN:QFN-56-1EP_7x7mm_P0.4mm_EP3.2x3.2mm, symbol MCU_RaspberryPi:RP2040
- added U3: LIS2DH, Package_LGA:LGA-14_2x2mm_P0.35mm_LayoutBorder3x4y, symbol Sensor_Motion:LIS2DH
- C1: value 100nF -> 33pF; LCSC Part # C1525 -> (none)
- C11: value 1uF -> 100nF; LCSC Part # C52923 -> (none)
- C12, C15, C16, C4: LCSC Part # C1525 -> (none)
- C14: LCSC Part # C1525 -> (none); now not fitted
- C21: value 1uF -> 100uF; footprint Capacitor_SMD:C_0402_1005Metric -> (none); LCSC Part # C52923 -> (none); now not fitted
- C5: value 6.8pF -> 100nF; LCSC Part # C1576 -> (none)
- C6: value 6.8pF -> 1uF; LCSC Part # C1576 -> (none)
- C8: value 68pF -> 1uF; LCSC Part # C389103 -> (none)
- J2: renamed from J3; LCSC Part # C3020560 -> C165948
- R4: value 10k -> 27.4R; LCSC Part # C25744 -> (none)
- SW1: value SW_Push -> RESET; footprint Button_Switch_SMD:SW_SPST_TS-1088-xR025 -> Button_Switch_SMD:SW_Push_SPST_NO_Alps_SKRK; LCSC Part # C720477 -> (none)
- SW3: renamed from SW2; footprint Button_Switch_THT:SW_PUSH-12mm -> Button_Switch_THT:SW_PUSH_6mm
- SW4: renamed from SW3; footprint Button_Switch_THT:SW_PUSH-12mm -> Button_Switch_THT:SW_PUSH_6mm
- SW5: renamed from SW4; footprint Button_Switch_THT:SW_PUSH-12mm -> Button_Switch_THT:SW_PUSH_6mm
- SW6: renamed from SW5; footprint Button_Switch_THT:SW_PUSH-12mm -> Button_Switch_THT:SW_PUSH_6mm
- Y1: value 32MHz -> 12MHz; LCSC (none) -> C9002; LCSC Part # C5441424 -> (none)
- renumbered C2 to C22, C3 to C23, C10 to C24, C9 to C25, C20 to C26, C22 to C27, C24 to C28, C25 to C29, C26 to C30, C27 to C31, C28 to C32, C29 to C33, C30 to C34, C31 to C35, C32 to C36, C33 to C37, C42 to C38, C19 to C39, C46 to C40, C47 to C41, D2 to D10, D3 to D11, D4 to D3, D7 to D6, D1 to D9, J4 to J3, J1 to J4, L6 to L1, L3 to L2, Q3 to Q1, R2 to R1, R9 to R10, R6 to R11, R7 to R12, R12 to R13, R13 to R14, R8 to R9, TP3 to TP2, TP5 to TP3, TP2 to TP4, TP4 to TP5, U1 to U4, U4 to U5, U8 to U6
Connections:
- net CTRL is gone; now on net D-: R4.1
- net VR_PA is gone; now on net GND: C8.2
- net +3V3: now also C12.1, C16.1, C4.1, C8.1, C10.1, C13.1, C7.1, C9.1, J1.1 (Pin_1), R2.1, R6.1, U1.8 (VCC), U2.1 (IOVDD), U2.10 (IOVDD), U2.22 (IOVDD), U2.33 (IOVDD), U2.42 (IOVDD), U2.43 (ADC_AVDD), U2.44 (VREG_VIN), U2.48 (USB_VDD), U2.49 (IOVDD), U3.8 (Vdd); no longer C1.1, C14.1
- net BUSY: now also U2.30 (GPIO19)
- net CS: now also U2.27 (GPIO16), U3.4 (~{CS})
- net D+: now also R5.1
- net DC: now also U2.28 (GPIO17)
- net GND: now also C1.1, C12.2, C4.2, C5.2, C6.2, AE2.0 (Shield), C10.2, C13.2, C2.1, C3.2, C7.2, C9.2, D1.1 (VSS), D12.1 (VSS), D13.1 (VSS), D14.1 (VSS), D15.1 (VSS), D16.1 (VSS), D2.1 (VSS), D20.1 (VSS), D21.1 (VSS), D4.1 (VSS), D5.1 (VSS), D7.1 (VSS), H1.1, H2.1, J1.2 (Pin_2), SW10.2, SW2.1, SW7.2, SW8.2, SW9.2, U1.4 (GND), U2.19 (TESTEN), U2.31 (GPIO20), U2.57 (GND), U3.10 (GND), U3.11 (GND), U3.12 (GND), U3.13 (GND), U3.14 (GND), U3.9 (GND); no longer C1.2, C12.1, C4.1, C5.1, C6.1, C8.1, R4.2
- net RST: now also U2.29 (GPIO18)
- net SPI_MOSI: now also U2.14 (GPIO11)
- net SPI_SCK: now also U2.13 (GPIO10)
- net SWCLK: now also U2.24 (SWCLK)
- net SWDIO: now also U2.25 (SWDIO)
- net UART1_RX: now also U2.37 (GPIO25)
- net UART1_TX: now also U2.36 (GPIO24)
- net at SW1.2: now also R2.2, U2.26 (RUN); no longer C4.2
- net at Y1.3: now also C2.2, R3.1; no longer C6.2
- net at U4.21 (ANT): now also AE2.1 (A)
- net at Y1.1: now also C1.2, U2.20 (XIN); no longer C5.2
- net PB3 renamed BTN1
- net BTN1: now also U2.17 (GPIO14)
- net PB4 renamed BTN2
- net BTN2: now also U2.18 (GPIO15)
- net PB5 renamed BTN3
- net BTN3: now also U2.15 (GPIO12)
- net PB8 renamed BTN4
- net BTN4: now also U2.16 (GPIO13)
- net PC13 renamed BUZ
- net BUZ: now also U2.35 (GPIO23)
- removed net VFBSMPS: C12.2, C16.1
- new net: D12.2 (DIN), D21.4 (DOUT), D7.2 (DIN)
- new net: D12.4 (DOUT), D13.2 (DIN), D14.2 (DIN)
- new net: D1.2 (DIN), D2.2 (DIN), R8.2
- new net: R3.2, U2.21 (XOUT)
- new net: D15.2 (DIN), D16.2 (DIN), D2.4 (DOUT)
- new net: R7.1, SW2.2
- new net: C14.1, U3.7 (Vdd_IO)
- new net: D16.4 (DOUT), D4.2 (DIN), D5.2 (DIN)
- new net: R4.2, U2.46 (USB_DM)
- new net: R5.2, U2.47 (USB_DP)
- new net +1V1: C3.1, C5.1, C6.1, U2.23 (DVDD), U2.45 (VREG_VOUT), U2.50 (DVDD)
- new net BTN5: SW7.1, U2.4 (GPIO2)
- new net BTN6: SW8.1, U2.2 (GPIO0)
- new net BTN7: SW9.1, U2.3 (GPIO1)
- new net BTN8: SW10.1, U2.5 (GPIO3)
- new net DOUT: D20.2 (DIN), D21.2 (DIN), D5.4 (DOUT)
- new net GPIO4: J1.6 (Pin_6), U2.6 (GPIO4)
- new net GPIO5: J1.5 (Pin_5), U2.7 (GPIO5)
- new net GPIO9: R8.1
- new net QSPI_SCK: U1.6 (CLK), U2.52 (QSPI_SCLK)
- new net QSPI_SD0: U1.5 (DI/IO_{0}), U2.53 (QSPI_SD0)
- new net QSPI_SD1: U1.2 (DO/IO_{1}), U2.55 (QSPI_SD1)
- new net QSPI_SD2: U1.3 (~{WP}/IO_{2}), U2.54 (QSPI_SD2)
- new net QSPI_SD3: U1.7 (~{HOLD}/~{RESET}/IO_{3}), U2.51 (QSPI_SD3)
- new net QSPI_SS: R6.2, R7.2, U1.1 (~{CS}), U2.56 (~{QSPI_SS})
- new net SCL: J1.3 (Pin_3), U2.12 (GPIO9), U3.1 (SCL/SPC)
- new net SDA: J1.4 (Pin_4), U2.11 (GPIO8), U3.2 (SDA/SDI)
- new net SDO: U3.3 (SDO)
- new net VDD: D1.3 (VDD), D12.3 (VDD), D13.3 (VDD), D14.3 (VDD), D16.3 (VDD), D2.3 (VDD), D20.3 (VDD), D21.3 (VDD), D4.3 (VDD), D5.3 (VDD), D7.3 (VDD)
- no-connect marks 52 -> 31
Other:
- removed sheet ledblock
- removed sheet ledblock1
- removed sheet ledblock2
- note added: "Accelerometer"
- note added: "For fun"
- note added: "Mounting Holes"
- note added: "RP2040 MCU"
- note added: "Removed to lower BOM"
- note added: "SAO"
- note added: "USB-C"
- note removed: "17dBm to stay under the limit of 19dBm"
- note removed: "CN470 (470-510 MHz)"
- note removed: "Configure power output to 16/17dBm in firmware (VDDPA)"
- note removed: "RF Output"
- note removed: "Removed to lower BOM cost"
- note removed: "STM32 MCU"
- moved on the sheet: BZ1, C22, C23, C24, C25, C26, C27, C28, C29, C30, C31, C32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

Commit message: final board for prod
Parts:
- added R16, R17: 4k7, Resistor_SMD:R_0402_1005Metric, symbol Device:R
- AE2: now not fitted
- C1, C2: LCSC Part # (none) -> C1562
- C10, C11, C12, C13, C15, C16, C3, C4, C5: LCSC Part # (none) -> C1525
- C39: now in the parts list
- C6, C8: LCSC Part # (none) -> C52923
- D8: LCSC Part # C84256 -> C84264
- L1: LCSC Part # C354558 -> C2047322
- R15: value 3.3k -> 2.2k; LCSC Part # C25890 -> C25879
- R2, R6: LCSC Part # (none) -> C25744
- R4, R5: LCSC Part # (none) -> C274349
- SW1, SW2: footprint Button_Switch_SMD:SW_Push_SPST_NO_Alps_SKRK -> footprints:KEY-SMD_K2-1177SW-A4DW-06; LCSC Part # (none) -> C92582
- U1: LCSC Part # (none) -> C179173
- U2: LCSC Part # (none) -> C2040
- Y1: LCSC Part # (none) -> C9002
Connections:
- net +3V3: now also R16.1, R17.1
- net SCL: now also R17.2
- net SDA: now also R16.2
- net VDD: now also D15.3 (VDD)
- no-connect marks 31 -> 39
Other:
- note added: "For fun, not mounting"
- note added: "for ~540mA charge current"
- note removed: "For fun"
- note removed: "for ~300mA charge current"
