File: hardware/ledblock.kicad_sch (KiCad schematic)
At the start: 2 parts

Commit message: final fixes
Parts:
- D10, D11: now not fitted; now left out of the parts list
Changed lines of the file:
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@@
 		(unit 1)
 		(exclude_from_sim no)
-		(in_bom yes)
-		(on_board yes)
-		(dnp no)
+		(in_bom no)
+		(on_board no)
+		(dnp yes)
 		(fields_autoplaced yes)
 		(property "Reference" "D11"
@@
 		(unit 1)
 		(exclude_from_sim no)
-		(in_bom yes)
-		(on_board yes)
-		(dnp no)
+		(in_bom no)
+		(on_board no)
+		(dnp yes)
 		(fields_autoplaced yes)
 		(property "Reference" "D10"

Commit message: add v2 w/o lora
Parts:
- D12: renamed from D10; now fitted; now in the parts list
- D13: renamed from D11; now fitted; now in the parts list
Changed lines of the file:
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@@
 		(dnp no)
 		(fields_autoplaced yes)
-		(property "Reference" "#PWR081"
+		(property "Reference" "#PWR083"
 			(at 147.32 109.22 0)
 			(effects
@@
 		(instances
 			(project "falloutbadge"
-				(path "/1a4a4e67-d7d1-492f-96ac-ef94582179fd/2fe96ec9-bc57-4c96-8b9a-7c7b8976d9a5"
-					(reference "#PWR089")
-					(unit 1)
-				)
-				(path "/1a4a4e67-d7d1-492f-96ac-ef94582179fd/ca2642aa-8349-4fc9-9750-554b8e7f584a"
-					(reference "#PWR081")
-					(unit 1)
-				)
-				(path "/1a4a4e67-d7d1-492f-96ac-ef94582179fd/f28209f4-aebd-4921-8505-b2d277a085e6"
-					(reference "#PWR085")
+				(path "/1a4a4e67-d7d1-492f-96ac-ef94582179fd/38bf4992-64ba-4b08-abc7-132b243ca13c"
+					(reference "#PWR095")
+					(unit 1)
+				)
+				(path "/1a4a4e67-d7d1-492f-96ac-ef94582179fd/c6b4f9a6-3882-46e8-971a-f0b60669210d"
+					(reference "#PWR083")
+					(unit 1)
+				)
+				(path "/1a4a4e67-d7d1-492f-96ac-ef94582179fd/cc1ade73-4512-43da-b58c-81be713da4ab"
+					(reference "#PWR091")
+					(unit 1)
+				)
+				(path "/1a4a4e67-d7d1-492f-96ac-ef94582179fd/eb4f4b5a-d289-4af8-930b-5b7032848f03"
+					(reference "#PWR087")
 					(unit 1)
 				)
@@
 		(unit 1)
 		(exclude_from_sim no)
-		(in_bom no)
-		(on_board no)
-		(dnp yes)
-		(fields_autoplaced yes)
-		(property "Reference" "D11"
+		(in_bom yes)
+		(on_board yes)
+		(dnp no)
+		(fields_autoplaced yes)
+		(property "Reference" "D13"
 			(at 170.18 101.2346 90)
 			(effects
@@
 		(instances
 			(project "falloutbadge"
-				(path "/1a4a4e67-d7d1-492f-96ac-ef94582179fd/2fe96ec9-bc57-4c96-8b9a-7c7b8976d9a5"
+				(path "/1a4a4e67-d7d1-492f-96ac-ef94582179fd/38bf4992-64ba-4b08-abc7-132b243ca13c"
+					(reference "D19")
+					(unit 1)
+				)
+				(path "/1a4a4e67-d7d1-492f-96ac-ef94582179fd/c6b4f9a6-3882-46e8-971a-f0b60669210d"
+					(reference "D13")
+					(unit 1)
+				)
+				(path "/1a4a4e67-d7d1-492f-96ac-ef94582179fd/cc1ade73-4512-43da-b58c-81be713da4ab"
+					(reference "D17")
+					(unit 1)
+				)
+				(path "/1a4a4e67-d7d1-492f-96ac-ef94582179fd/eb4f4b5a-d289-4af8-930b-5b7032848f03"
 					(reference "D15")
-					(unit 1)
-				)
-				(path "/1a4a4e67-d7d1-492f-96ac-ef94582179fd/ca2642aa-8349-4fc9-9750-554b8e7f584a"
-					(reference "D11")
-					(unit 1)
-				)
-				(path "/1a4a4e67-d7d1-492f-96ac-ef94582179fd/f28209f4-aebd-4921-8505-b2d277a085e6"
-					(reference "D13")
 					(unit 1)
 				)
@@
 		(dnp no)
 		(fields_autoplaced yes)
-		(property "Reference" "#PWR080"
+		(property "Reference" "#PWR082"
 			(at 143.51 113.03 0)
 			(effects
@@
 		(instances
 			(project "falloutbadge"
-				(path "/1a4a4e67-d7d1-492f-96ac-ef94582179fd/2fe96ec9-bc57-4c96-8b9a-7c7b8976d9a5"
-					(reference "#PWR088")
-					(unit 1)
-				)
-				(path "/1a4a4e67-d7d1-492f-96ac-ef94582179fd/ca2642aa-8349-4fc9-9750-554b8e7f584a"
-					(reference "#PWR080")
-					(unit 1)
-				)
-				(path "/1a4a4e67-d7d1-492f-96ac-ef94582179fd/f28209f4-aebd-4921-8505-b2d277a085e6"
-					(reference "#PWR084")
+				(path "/1a4a4e67-d7d1-492f-96ac-ef94582179fd/38bf4992-64ba-4b08-abc7-132b243ca13c"
+					(reference "#PWR094")
+					(unit 1)
+				)
+				(path "/1a4a4e67-d7d1-492f-96ac-ef94582179fd/c6b4f9a6-3882-46e8-971a-f0b60669210d"
+					(reference "#PWR082")
+					(unit 1)
+				)
+				(path "/1a4a4e67-d7d1-492f-96ac-ef94582179fd/cc1ade73-4512-43da-b58c-81be713da4ab"
+					(reference "#PWR090")
+					(unit 1)
+				)
+				(path "/1a4a4e67-d7d1-492f-96ac-ef94582179fd/eb4f4b5a-d289-4af8-930b-5b7032848f03"
+					(reference "#PWR086")
 					(unit 1)
 				)
@@
 		(dnp no)
 		(fields_autoplaced yes)
-		(property "Reference" "#PWR079"
+		(property "Reference" "#PWR081"
 			(at 115.57 109.22 0)
 			(effects
@@
 		(instances
 			(project "falloutbadge"
-				(path "/1a4a4e67-d7d1-492f-96ac-ef94582179fd/2fe96ec9-bc57-4c96-8b9a-7c7b8976d9a5"
-					(reference "#PWR087")
-					(unit 1)
-				)
-				(path "/1a4a4e67-d7d1-492f-96ac-ef94582179fd/ca2642aa-8349-4fc9-9750-554b8e7f584a"
-					(reference "#PWR079")
-					(unit 1)
-				)
-				(path "/1a4a4e67-d7d1-492f-96ac-ef94582179fd/f28209f4-aebd-4921-8505-b2d277a085e6"
-					(reference "#PWR083")
+				(path "/1a4a4e67-d7d1-492f-96ac-ef94582179fd/38bf4992-64ba-4b08-abc7-132b243ca13c"
+					(reference "#PWR093")
+					(unit 1)
+				)
+				(path "/1a4a4e67-d7d1-492f-96ac-ef94582179fd/c6b4f9a6-3882-46e8-971a-f0b60669210d"
+					(reference "#PWR081")
+					(unit 1)
+				)
+				(path "/1a4a4e67-d7d1-492f-96ac-ef94582179fd/cc1ade73-4512-43da-b58c-81be713da4ab"
+					(reference "#PWR089")
+					(unit 1)
+				)
+				(path "/1a4a4e67-d7d1-492f-96ac-ef94582179fd/eb4f4b5a-d289-4af8-930b-5b7032848f03"
+					(reference "#PWR085")
 					(unit 1)
 				)
@@
 		(unit 1)
 		(exclude_from_sim no)
-		(in_bom no)
-		(on_board no)
-		(dnp yes)
-		(fields_autoplaced yes)
-		(property "Reference" "D10"
+		(in_bom yes)
+		(on_board yes)
+		(dnp no)
+		(fields_autoplaced yes)
+		(property "Reference" "D12"
 			(at 138.43 101.2346 90)
 			(effects
@@
 		(instances
 			(project "falloutbadge"
-				(path "/1a4a4e67-d7d1-492f-96ac-ef94582179fd/2fe96ec9-bc57-4c96-8b9a-7c7b8976d9a5"
+				(path "/1a4a4e67-d7d1-492f-96ac-ef94582179fd/38bf4992-64ba-4b08-abc7-132b243ca13c"
+					(reference "D18")
+					(unit 1)
+				)
+				(path "/1a4a4e67-d7d1-492f-96ac-ef94582179fd/c6b4f9a6-3882-46e8-971a-f0b60669210d"
+					(reference "D12")
+					(unit 1)
+				)
+				(path "/1a4a4e67-d7d1-492f-96ac-ef94582179fd/cc1ade73-4512-43da-b58c-81be713da4ab"
+					(reference "D16")
+					(unit 1)
+				)
+				(path "/1a4a4e67-d7d1-492f-96ac-ef94582179fd/eb4f4b5a-d289-4af8-930b-5b7032848f03"
 					(reference "D14")
-					(unit 1)
-				)
-				(path "/1a4a4e67-d7d1-492f-96ac-ef94582179fd/ca2642aa-8349-4fc9-9750-554b8e7f584a"
-					(reference "D10")
-					(unit 1)
-				)
-				(path "/1a4a4e67-d7d1-492f-96ac-ef94582179fd/f28209f4-aebd-4921-8505-b2d277a085e6"
-					(reference "D12")
 					(unit 1)
 				)
@@
 		(dnp no)
 		(fields_autoplaced yes)
-		(property "Reference" "#PWR082"
+		(property "Reference" "#PWR084"
 			(at 175.26 113.03 0)
 			(effects
@@
 		(instances
 			(project "falloutbadge"
-				(path "/1a4a4e67-d7d1-492f-96ac-ef94582179fd/2fe96ec9-bc57-4c96-8b9a-7c7b8976d9a5"
-					(reference "#PWR090")
-					(unit 1)
-				)
-				(path "/1a4a4e67-d7d1-492f-96ac-ef94582179fd/ca2642aa-8349-4fc9-9750-554b8e7f584a"
-					(reference "#PWR082")
-					(unit 1)
-				)
-				(path "/1a4a4e67-d7d1-492f-96ac-ef94582179fd/f28209f4-aebd-4921-8505-b2d277a085e6"
-					(reference "#PWR086")
-					(unit 1)
-				)
+				(path "/1a4a4e67-d7d1-492f-96ac-ef94582179fd/38bf4992-64ba-4b08-abc7-132b243ca13c"
+					(reference "#PWR096")
+					(unit 1)
+				)
+				(path "/1a4a4e67-d7d1-492f-96ac-ef94582179fd/c6b4f9a6-3882-46e8-971a-f0b60669210d"
+					(reference "#PWR084")
+					(unit 1)
+				)
+				(path "/1a4a4e67-d7d1-492f-96ac-ef94582179fd/cc1ade73-4512-43da-b58c-81be713da4ab"
+					(reference "#PWR092")
+					(unit 1)
+				)
+				(path "/1a4a4e67-d7d1-492f-96ac-ef94582179fd/eb4f4b5a-d289-4af8-930b-5b7032848f03"
+					(reference "#PWR088")
+					(unit 1)
+				)
